File: PCB_Files/watch.kicad_sch (KiCad schematic)
At the start: 39 parts, among them J1 USB_C_Receptacle_USB2.0_16P, Q1 BC847, Q2 BC847, SW1 SW_Push, U1 APS6404L-3SQRx-ZR, U2 ESP32-PICO-D4, U3 CP2102N-Axx-xQFN28, Y1 SG-3030CM

Commit message: Schematics Updated
Parts:
- added C17, C24: 1 uF, symbol Device:C
- added C19, C20, C21, C23: 10 uF, symbol Device:C
- added C22, C5: 0.1 uF, symbol Device:C
- added C25, C6, C7: 4.7 uF, symbol Device:C
- added C26: 0.01 uF, symbol Device:C
- added D5: LED, symbol Device:LED
- added Q3: FS8205A, symbol FS8205A:FS8205A
- added R13: 2.7k, symbol Device:R
- added R14, R15: 330, symbol Device:R
- added R16: 2k, symbol Device:R
- added R17: 0R, symbol Device:R
- added U10: LSM6DS3, Package_LGA:LGA-14_3x2.5mm_P0.5mm_LayoutBorder3x4y, symbol Sensor_Motion:LSM6DS3
- added U11: MAX-M10S, RF_GPS:ublox_MAX, symbol RF_GPS:MAX-M10S
- added U4: TPS7A0533PDBV, Package_TO_SOT_SMD:SOT-23-5, symbol Regulator_Linear:TPS7A0533PDBV
- added U5: MCP73831-2-OT, Package_TO_SOT_SMD:SOT-23-5, symbol Battery_Management:MCP73831-2-OT
- added U6: AP9101CK6, Package_TO_SOT_SMD:SOT-23-6, symbol Battery_Management:AP9101CK6
- added U7: MAX30105EFD_T, Library:14-OESIP, symbol MAX30105EFD_T:MAX30105EFD_T
- added U8: LIS2DH, Package_LGA:LGA-14_2x2mm_P0.35mm_LayoutBorder3x4y, symbol Sensor_Motion:LIS2DH
- added U9: MAX8510EXK33T, Library:SOT65P210X110-5N, symbol MAX8510EXK33T:MAX8510EXK33T
Connections:
- net +3V3: now also U10.5 (VDDIO), U10.8 (VDD), U11.7 (VCC_IO), U11.8 (VCC)
- net GND: now also C17.2, C19.2, C20.2, C21.1, C22.1, C23.1, C24.1, C25.2, C5.2, C6.2, C7.2, Q3.2, Q3.3, R16.1, U10.6 (GND), U10.7 (GND), U11.1 (GND), U11.10 (GND), U11.12 (GND), U4.2 (GND), U5.2 (V_{SS}), U6.6 (VSS), U7.12 (GND), U7.4 (PGND), U8.10 (GND), U8.11 (GND), U8.12 (GND), U8.13 (GND), U8.14 (GND), U8.9 (GND), U9.2 (GND)
- net VBUS: now also C6.1, D5.2 (A), U5.4 (V_{DD})
- new net: R15.1, U5.1 (STAT)
- new net: D5.1 (K), R15.2
- new net: C17.1, U4.1 (IN)
- new net: C22.2, C23.2, U8.8 (Vdd)
- new net: C20.1, R17.2
- new net: R16.2, U5.5 (PROG)
- new net: R17.1, U7.9 (VLED+)
- new net: C24.2, U9.1 (IN), U9.3 (~{SHDN})
- new net: C26.2, U9.4 (BP)
- new net: C19.1, U4.5 (OUT)
- new net: C21.2, U7.11 (VDD)
- new net: R13.2, U6.2 (VM)
- new net: Q3.4, U6.1 (DO)
- new net: Q3.5, U6.3 (CO)
- new net: Q3.1, Q3.8
- new net 3V3_U6: C25.1, C26.1, U9.5 (OUT)
- new net Batt+: C7.1, R14.1, U4.3 (EN), U5.3 (V_{BAT})
- new net C5: C5.1, R14.2, U6.5 (VDD)
- new net P-: Q3.6, Q3.7, R13.1
Other:
- moved on the sheet: C14, C4, R2, R3, SW1, U1, Y1

Commit message: Connected few peripherals and formatting
Parts:
- removed C24: 1 uF, symbol Device:C
- removed C25: 4.7 uF, symbol Device:C
- removed C26: 0.01 uF, symbol Device:C
- removed U9: MAX8510EXK33T, Library:SOT65P210X110-5N, symbol MAX8510EXK33T:MAX8510EXK33T
- added C27, C28, C29: 0.1 uF, symbol Device:C
- added C30, C31: 1uF, symbol Device:C
- added Q4, Q5: BSS138, Package_TO_SOT_SMD:SOT-23, symbol Transistor_FET:BSS138
- added R18, R19, R20, R21: 4.7k, symbol Device:R
- added U12: MCP1700x-120xxMB, Package_TO_SOT_SMD:SOT-89-3, symbol Regulator_Linear:MCP1700x-120xxMB
Connections:
- net +3V3: now also R17.1, U7.9 (VLED+), C27.1, C28.2
- net GND: now also U10.2 (SDX), U10.3 (SCX), C27.2, C28.1, C29.1, C30.1, C31.1, U12.1 (GND)
- net MISO: now reaches U10.1 (SDO/SA0)
- net MISO: now also U2.28 (SD2/IO9), U8.3 (SDO)
- net CS: now reaches U10.12 (CS)
- net CS: now also U2.21 (IO15), U8.4 (~{CS})
- net SCL: now reaches U10.13 (SCL)
- net SCL: now also U2.34 (IO5), U8.1 (SCL/SPC)
- net MOSI: now reaches U10.14 (SDA)
- net MOSI: now also U2.29 (SD3/IO10), U8.2 (SDA/SDI)
- net INTR1_IMU: now reaches U10.4 (INT1)
- net INTR1_IMU: now also U2.24 (IO4)
- net INTR2_IMU: now reaches U10.9 (INT2)
- net INTR2_IMU: now also U2.22 (IO2)
- net SDA: now reaches U2.14 (IO25)
- net SDA: now also R21.2
- net SCL_i2c: now reaches U2.27 (IO17)
- net SCL_i2c: now also R18.2
- net at U8.7 (Vdd_IO): now also C22.2, C23.2, U8.8 (Vdd)
- net 3V3: now reaches C19.1, U4.5 (OUT)
- net 3V3: now also C30.2, U12.2 (VI)
- net at C21.2, U7.11 (VDD): now also C29.2
- net LV_SCL: now reaches U7.2 (SCL)
- net LV_SCL: now also Q4.2 (S), R20.1
- net LV_SDA: now reaches U7.3 (SDA)
- net LV_SDA: now also Q5.2 (S), R19.1
- new net: Q5.3 (D), R21.1
- new net: Q4.3 (D), R18.1
- new net 1.8V: C31.2, Q4.1 (G), Q5.1 (G), R19.2, R20.2, U12.3 (VO)
- no-connect marks 0 -> 3
Other:
- note added: "Accelerometer"
- note added: "Battery Management"
- note added: "Battery Protection Module"
- note added: "Charging Module"
- note added: "Converts 3.3V to 1.8V"
- note added: "Converts 3.7V to 3.3V"
- note added: "Crystal Oscillator"
- note added: "GNSS Receiver (Incomplete)"
- note added: "IMU"
- note added: "MCU"
- note added: "Optical Sensor (Incomplete)"
- note added: "Peripherals"
- note added: "SPI/QPI PSRAM"
- note added: "Serial Boot&Switch"
- note added: "Smart Watch"
- note added: "Type-C Port"
- note added: "USB to TTL(Serial)Convertor"
- note added: "Voltage Regulator"
- moved on the sheet: C1, C10, C11, C12, C13, C14, C15, C16, C17, C18, C19, C2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

Commit message: Added Sensors
Parts:
- added C24, C25: 1 uF, symbol Device:C
- added U13: DRV2605LDGS, Package_SO:VSSOP-10_3x3mm_P0.5mm, symbol Driver_Haptic:DRV2605LDGS
- added U9: BMP388, symbol BMP388:BMP388
Connections:
- net +3V3: now also C24.1, U13.10 (VDD), U13.5 (EN), U13.6 (VDD/NC), U9.1 (VDDIO), U9.10 (VDD)
- net 1.8V: now also R20.1; no longer R20.2
- net GND: now also C24.2, C25.2, U13.4 (IN/TRIG), U13.8 (GND), U9.3 (VSS), U9.8 (VSS), U9.9 (VSS)
- net LV_SCL: now also R20.2, U13.2 (SCL); no longer R20.1
- net LV_SDA: now also U13.3 (SDA)
- new net: C25.1, U13.1 (REG)
- new net Motor_OUT+: U13.7 (OUT+)
- new net Motor_OUT-: U13.9 (OUT-)
Other:
- note added: "Barometer (incomplete)"
- note added: "DRV2605L"
- note added: "I2C Lines"
- moved on the sheet: C20, C21, C22, C23, C27, C28, C29, Q4, Q5, R17, R18, R19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

Commit message: Added Connections for Barometer, GNSS, Optical Sensor
Parts:
- added AE1: Antenna_Shield, symbol Device:Antenna_Shield
- added C26: 47 pF, symbol Device:C
- added D10, D11, D12, D7, D8, D9: LED, symbol Device:LED
- added D6: PESD0402-0402T, Diode_SMD:D_SOD-923, symbol Diode:ESD9B3.3ST5G
- added FB1: FerriteBead, symbol Device:FerriteBead
- added Q6, Q7: BSS138, Package_TO_SOT_SMD:SOT-23, symbol Transistor_FET:BSS138
- added R22, R23, R24, R25, R29: 10k, symbol Device:R
- added R26, R27, R28: 33, symbol Device:R
- added R30: 0R, symbol Device:R
Connections:
- net +3V3: now also U11.15 (VIO_SEL), U11.6 (V_BCKP), U9.6 (CSB), Q6.1 (G), Q7.1 (G), R22.1, R23.1, R24.1, R25.1, R29.1
- net 1.8V: now also C21.2, C29.2, U7.11 (VDD)
- net GND: now also AE1.2 (Shield), C26.2, D6.1 (A1)
- net LV_SCL: no longer U13.2 (SCL)
- net LV_SDA: no longer U13.3 (SDA)
- net SCL_i2c: now also Q6.2 (S), R24.2
- net SDA: now also Q7.2 (S), R25.2
- net at U11.11 (RF_IN): now also AE1.1 (A), D6.2 (A2), FB1.1
- net at U11.14 (VCC_RF): now also R28.1
- net at U11.16 (SDA): now also R26.2
- net at U11.17 (SCL): now also R27.2
- net at U11.9 (~{RESET}): now also R29.2
- net at C20.1, R17.2: now also R30.2
- net SCL_i2c_R: now reaches U9.2 (SCK)
- net SCL_i2c_R: now also U13.2 (SCL), Q6.3 (D), R22.2, R27.1
- net SDA_R: now reaches U9.4 (SDI)
- net SDA_R: now also U13.3 (SDA), Q7.3 (D), R23.2, R26.1
- net R_DRV: now reaches U7.5 (R_DRV)
- net R_DRV: now also D7.1 (K), D8.1 (K)
- net IR_DRV: now reaches U7.6 (IR_DRV)
- net IR_DRV: now also D10.1 (K), D9.1 (K)
- net G_DRV: now reaches U7.7 (G_DRV)
- net G_DRV: now also D11.1 (K), D12.1 (K)
- new net VCC_RF: C26.1, FB1.2, R28.2
- new net VLED+_EX: D10.2 (A), D11.2 (A), D12.2 (A), D7.2 (A), D8.2 (A), D9.2 (A), R30.1
- no-connect marks 3 -> 11
Other:
- note added: "Barometer"
- note added: "GNSS Receiver"
- note added: "I2C for Optical Sensor"
- note added: "Optical Sensor"
- note removed: "Barometer (incomplete)"
- note removed: "GNSS Receiver (Incomplete)"
- note removed: "Optical Sensor (Incomplete)"
- moved on the sheet: C20, C21, C24, C25, C29, Q4, Q5, R17, R18, R19, R20, R21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

Commit message: Schematics Completed
Parts:
- added AE2: Antenna_Shield, symbol Device:Antenna_Shield
- added C32: 1 uF, symbol Device:C
- added C33, C37, C39: 0.1 uF, symbol Device:C
- added C34: 0.1 uF, Capacitor_SMD:C_0805_2012Metric_Pad1.18x1.45mm_HandSolder, symbol Device:C
- added C35: 1.2 pF, symbol Device:C
- added C36: 1.5 pF, symbol Device:C
- added C38: 0.1uF, Capacitor_SMD:C_0805_2012Metric_Pad1.18x1.45mm_HandSolder, symbol Device:C
- added D13, D14: LED, LED_SMD:LED_0805_2012Metric_Pad1.15x1.40mm_HandSolder, symbol Device:LED
- added D15: D_Zener, Diode_SMD:D_0805_2012Metric_Pad1.15x1.40mm_HandSolder, symbol Device:D_Zener
- added J2: Conn_01x15_MountingPin, symbol Connector_Generic_MountingPin:Conn_01x15_MountingPin
- added J3: Conn_01x02_Pin, symbol Connector:Conn_01x02_Pin
- added L2: 1.8 nH, symbol Device:L
- added Q8: BC847, Package_TO_SOT_SMD:SOT-23, symbol Transistor_BJT:BC847
- added R31: 10k, Resistor_SMD:R_0805_2012Metric_Pad1.20x1.40mm_HandSolder, symbol Device:R
- added R32, R33: 0.3k, Resistor_SMD:R_0805_2012Metric_Pad1.20x1.40mm_HandSolder, symbol Device:R
- added R34: 22.1k, Resistor_SMD:R_0805_2012Metric_Pad1.20x1.40mm_HandSolder, symbol Device:R
- added R35: 47.5k, Resistor_SMD:R_0805_2012Metric_Pad1.20x1.40mm_HandSolder, symbol Device:R
- added R36: 22, Resistor_SMD:R_0805_2012Metric_Pad1.20x1.40mm_HandSolder, symbol Device:R
- added R37: 1k, Resistor_SMD:R_0805_2012Metric_Pad1.20x1.40mm_HandSolder, symbol Device:R
- added R38, R39, R40, R41: 10k, symbol Device:R
- added U14: W25Q64JVSSIQ, Library:SOIC-8_5P28X5P28_WIN, symbol 2026-01-31_10-07-27:W25Q64JVSSIQ
- C12: value NC -> 0 F
- C18: value 100nF -> 4.7 uF; footprint Capacitor_SMD:C_0805_2012Metric -> Capacitor_SMD:C_0805_2012Metric_Pad1.18x1.45mm_HandSolder
- FB1: footprint (none) -> Inductor_SMD:L_0805_2012Metric_Pad1.05x1.20mm_HandSolder
- J1: footprint (none) -> Connector_USB:USB_C_Receptacle_HRO_TYPE-C-31-M-12
- Q3: footprint (none) -> Library:SOP65P640X120-8N
- R1: value NC -> 0R
- U9: footprint (none) -> Library:PQFN50P200X200X80-10N
Connections:
- net +3V3 is gone; now on net 3V3: C1.1, C10.1, C11.1, C12.1, C13.1, C2.1, C24.1, C27.1, C28.2, C3.1, C4.1, C9.1, D1.2 (A2), L1.2, Q6.1 (G), Q7.1 (G), R1.1, R17.1, R2.2, R22.1, R23.1, R24.1, R25.1, R29.1, U1.8 (VDD), U10.5 (VDDIO), U10.8 (VDD), U11.15 (VIO_SEL), U11.6 (V_BCKP), U11.7 (VCC_IO), U11.8 (VCC), U13.10 (VDD), U13.5 (EN), U13.6 (VDD/NC), U2.1 (VDDA), U2.19 (VDD3P3_RTC), U2.37 (VDD3P3_CPU), U2.43 (VDDA), U2.46 (VDDA), U7.9 (VLED+), U9.1 (VDDIO), U9.10 (VDD), U9.6 (CSB), Y1.1 (VIO), Y1.4 (Vcc)
- net 3V3: now also C18.2, C22.2, C23.2, R4.1, U3.6 (VDD), U3.7 (VREGIN), U8.7 (Vdd_IO), U8.8 (Vdd), C32.1, C33.2, C34.2, C37.1, C39.2, J2.10 (Pin_10), J2.3 (Pin_3), J2.4 (Pin_4), R38.2, R39.2, U14.8 (VCC)
- net Batt+: now also C17.1, U4.1 (IN), D15.1 (K)
- net CE: now also U2.24 (IO4)
- net CS: now also J2.6 (Pin_6)
- net GND: now also Q3.1, Q3.8, AE2.2 (Shield), C32.2, C33.1, C34.1, C35.2, C36.2, C37.2, C38.1, C39.1, J2.1 (Pin_1), J2.11 (Pin_11), J2.MP (MountPin), Q8.2 (E), R31.1, R35.1, R40.1, R41.1, U14.4 (GND)
- net INTR1_IMU: now also U2.10 (IO34), R39.1; no longer U2.24 (IO4)
- net MOSI: now also J2.8 (Pin_8)
- net Motor_OUT+: now also J3.1 (Pin_1)
- net Motor_OUT-: now also J3.2 (Pin_2)
- net SCL: now also J2.7 (Pin_7)
- net SCL_i2c_R: now also J2.15 (Pin_15)
- net SDA_R: now also J2.14 (Pin_14)
- net VBUS: now also D15.2 (A), R32.2, R33.1, R34.1; no longer R4.1, U3.7 (VREGIN), U3.8 (VBUS)
- net VSPICLK: now also U14.6 (CLK)
- net VSPID: now also U14.5 (DI(IO0))
- net VSPIHD: now also U14.7 (/HOLD_OR_/RESET(IO3))
- net VSPIQ: now also U14.2 (DO(IO1))
- net VSPIWP: now also U14.3 (/WP(IO2))
- net CTP_INT: now reaches U2.11 (IO35)
- net CTP_INT: now also J2.13 (Pin_13), R38.1
- net RS: now reaches U2.13 (IO33)
- net RS: now also J2.5 (Pin_5)
- net RST: now reaches U2.15 (IO26)
- net RST: now also J2.9 (Pin_9)
- net BL_PWM: now reaches U2.16 (IO27)
- net BL_PWM: now also R37.1
- net CTP_RST: now reaches U2.17 (IO14)
- net CTP_RST: now also J2.12 (Pin_12)
- net LNA_IN: now reaches U2.2 (LNA_IN)
- net LNA_IN: now also C35.1, L2.1
- net CS_ROM: now reaches U2.20 (IO13)
- net CS_ROM: now also U14.1 (/CS)
- net at U2.26 (VDD_SDIO): now also C38.2
- net BTN1: now reaches U2.5 (SENSOR_VP)
- net BTN1: now also R40.2
- net BTN2: now reaches U2.8 (SENSOR_VN)
- net BTN2: now also R41.2
- net ACTIVE: now reaches U3.11 (~{SUSPEND})
- net ACTIVE: now also R31.2
- net at U3.18 (~{RXT}/GPIO.1): now also D14.1 (K)
- net at U3.19 (~{TXT}/GPIO.0): now also D13.1 (K)
- new net: D13.2 (A), R32.1
- new net: Q8.1 (B), R37.2
- new net: Q8.3 (C), R36.1
- new net: D14.2 (A), R33.2
- new net: AE2.1 (A), C36.1, L2.2
- new net: R34.2, R35.2, U3.8 (VBUS)
- new net LEDK: J2.2 (Pin_2), R36.2
- no-connect marks 11 -> 32
Other:
- note added: "Antenna of MCU"
- note added: "External Flash (8 MB)"
- note added: "Vibration Motor"
- note added: "ZIF Connector for Display"
- moved on the sheet: AE1, C1, C10, C11, C12, C13, C14, C15, C16, C17, C19, C2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

Commit message: Verified and corrected schematics
Parts:
- removed C22: 0.1 uF, symbol Device:C
- removed C23: 10 uF, symbol Device:C
- removed D3, D4: LED, symbol Device:LED
- removed R7, R8: 0.5k, symbol Device:R
- removed U14: W25Q64JVSSIQ, Library:SOIC-8_5P28X5P28_WIN, symbol 2026-01-31_10-07-27:W25Q64JVSSIQ
- removed U8: LIS2DH, Package_LGA:LGA-14_2x2mm_P0.35mm_LayoutBorder3x4y, symbol Sensor_Motion:LIS2DH
- added U8: W25Q128JVS, Package_SO:SOIC-8_5.23x5.23mm_P1.27mm, symbol Memory_Flash:W25Q128JVS
- C1, C10, C11, C12, C13, C14, C17, C19, C2, C20, C21, C24, C25, C26, C27, C28, C29, C3, C30, C31, C32, C33, C35, C36, C37, C39, C4, C5, C6, C7, C8, C9: footprint (none) -> Capacitor_SMD:C_0603_1608Metric
- C15, C16: footprint Capacitor_SMD:C_0805_2012Metric -> Capacitor_SMD:C_0603_1608Metric
- C18, C34, C38: footprint Capacitor_SMD:C_0805_2012Metric_Pad1.18x1.45mm_HandSolder -> Capacitor_SMD:C_0603_1608Metric
- D10, D11, D12, D5, D7, D8, D9: footprint (none) -> LED_SMD:LED_0603_1608Metric
- D13, D14: footprint LED_SMD:LED_0805_2012Metric_Pad1.15x1.40mm_HandSolder -> LED_SMD:LED_0603_1608Metric
- D15: footprint Diode_SMD:D_0805_2012Metric_Pad1.15x1.40mm_HandSolder -> Diode_SMD:D_0603_1608Metric
- J3: footprint (none) -> Diode_SMD:D_0603_1608Metric
- R1, R10, R11, R12, R13, R14, R15, R16, R17, R18, R19, R2, R20, R21, R22, R23, R24, R25, R26, R27, R28, R29, R3, R30, R38, R39, R4, R40, R41, R5, R6, R9: footprint (none) -> Resistor_SMD:R_0603_1608Metric
- R31, R32, R33, R34, R35, R36, R37: footprint Resistor_SMD:R_0805_2012Metric_Pad1.20x1.40mm_HandSolder -> Resistor_SMD:R_0603_1608Metric
- SW1: footprint (none) -> Button_Switch_SMD:SW_Push_SPST_NO_Alps_SKRK
Connections:
- net 3V3: now also R32.2, R33.1, U8.8 (VCC)
- net CS_ROM: now also U8.1 (~{CS})
- net DTR: now also Q1.3 (C); no longer Q1.2 (E)
- net GPIO0: now also Q1.2 (E); no longer Q1.3 (C)
- net VBUS: no longer R32.2, R33.1
- net VSPICLK: now also U8.6 (CLK)
- net VSPID: now also U8.5 (DI(IO0))
- net VSPIHD: now also U8.7 (IO3)
- net VSPIQ: now also U8.2 (DO(IO1))
- net VSPIWP: now also U8.3 (IO2)
- no-connect marks 32 -> 30
Other:
- note added: "External Flash (16 MB)"
- note removed: "Accelerometer"
- note removed: "External Flash (8 MB)"
- moved on the sheet: C15, C16, C39

Commit message: Added custom footprint library and assigned footprints
Parts:
- FB1: footprint Inductor_SMD:L_0805_2012Metric_Pad1.05x1.20mm_HandSolder -> Inductor_SMD:L_0603_1608Metric
- J2, L1, L2: footprint (none) -> Inductor_SMD:L_0603_1608Metric
- Q3: footprint Library:SOP65P640X120-8N -> footprints:SOP65P640X120-8N
- U7: footprint Library:14-OESIP -> footprints:14-OESIP
- U9: footprint Library:PQFN50P200X200X80-10N -> footprints:PQFN50P200X200X80-10N
Changed lines of the file:
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@@
 			)
 		)
-		(property "Footprint" ""
+		(property "Footprint" "Inductor_SMD:L_0603_1608Metric"
 			(at 419.1 304.8 0)
 			(effects
@@
 			)
 		)
-		(property "Footprint" "Inductor_SMD:L_0805_2012Metric_Pad1.05x1.20mm_HandSolder"
+		(property "Footprint" "Inductor_SMD:L_0603_1608Metric"
 			(at 315.722 306.07 90)
 			(effects
@@
 			)
 		)
-		(property "Footprint" ""
+		(property "Footprint" "Inductor_SMD:L_0603_1608Metric"
 			(at 105.41 218.44 0)
 			(effects
@@
 			)
 		)
-		(property "Footprint" "Library:PQFN50P200X200X80-10N"
+		(property "Footprint" "footprints:PQFN50P200X200X80-10N"
 			(at 99.06 298.45 0)
 			(effects
@@
 			)
 		)
-		(property "Footprint" "Library:14-OESIP"
+		(property "Footprint" "footprints:14-OESIP"
 			(at 161.29 303.53 0)
 			(effects
@@
 			)
 		)
-		(property "Footprint" ""
+		(property "Footprint" "Inductor_SMD:L_0603_1608Metric"
 			(at 107.95 55.88 0)
 			(effects
@@
 			)
 		)
-		(property "Footprint" "Library:SOP65P640X120-8N"
+		(property "Footprint" "footprints:SOP65P640X120-8N"
 			(at 344.17 199.39 0)
 			(effects

Commit message: Changes in schematics
Parts:
- removed D10, D11, D12, D13, D14, D7, D8, D9: LED, LED_SMD:LED_0603_1608Metric, symbol Device:LED
- removed D15: D_Zener, Diode_SMD:D_0603_1608Metric, symbol Device:D_Zener
- removed D2: SP0503BAHT, Package_TO_SOT_SMD:SOT-143, symbol Power_Protection:SP0503BAHT
- removed J1: USB_C_Receptacle_USB2.0_16P, Connector_USB:USB_C_Receptacle_HRO_TYPE-C-31-M-12, symbol Connector:USB_C_Receptacle_USB2.0_16P
- removed R5, R6: 5.1k, Resistor_SMD:R_0603_1608Metric, symbol Device:R
- added C22: 0.1 uF, Capacitor_SMD:C_0603_1608Metric, symbol Device:C
- added D13: SP0503BAHT, Package_TO_SOT_SMD:SOT-143, symbol Power_Protection:SP0503BAHT
- added D14: D_Zener, Diode_SMD:D_0603_1608Metric, symbol Device:D_Zener
- added D3, D4: LED, LED_SMD:LED_0603_1608Metric, symbol Device:LED
- added P1: USB_C_Plug_USB2.0, Connector_USB:USB_C_Receptacle_GCT_USB4125-xx-x-0190_6P_TopMnt_Horizontal, symbol Connector:USB_C_Plug_USB2.0
- added R7, R8: 330, Resistor_SMD:R_0603_1608Metric, symbol Device:R
- added SW2: SW_Push, Button_Switch_SMD:SW_Push_SPST_NO_Alps_SKRK, symbol Switch:SW_Push
- added TP1, TP2, TP3, TP4, TP5, TP6: TestPoint, TestPoint:TestPoint_Pad_D1.0mm, symbol Connector:TestPoint
- R3: value 0R -> 5.1k
- R32: value 0.3k -> 10k
- R33: value 0.3k -> 5.1k
Connections:
- net 1.8V: now also D4.2 (A), TP5.1
- net 3V3: now also D3.2 (A), TP4.1; no longer R33.1
- net Batt+: now also D14.1 (K), TP3.1
- net DTR: now also Q1.2 (E); no longer Q1.3 (C)
- net EN: now also C14.1, Q2.3 (C), R2.1, SW1.2; no longer R3.2
- net GND: now also R3.2, R33.2, C22.2, D13.1 (A), P1.A1 (GND), P1.A12 (GND), P1.B1 (GND), P1.B12 (GND), P1.S1 (SHIELD), R7.2, R8.2, SW2.1, TP6.1
- net GPIO0: now also Q1.3 (C), R32.1, C22.1, SW2.2; no longer Q1.2 (E)
- net U0RXD: now also TP1.1
- net VBUS: now also D13.4 (K), D14.2 (A), P1.A4 (VBUS), P1.A9 (VBUS), P1.B4 (VBUS), P1.B9 (VBUS)
- net G_DRV: no longer names the net of U7.7 (G_DRV)
- net IR_DRV: no longer names the net of U7.6 (IR_DRV)
- removed net RESET: C14.1, Q2.3 (C), R2.1, R3.1, SW1.2
- net R_DRV: no longer names the net of U7.5 (R_DRV)
- new net: P1.B5 (VCONN), R33.1
- new net: P1.A5 (CC), R3.1
- new net: D13.2 (K), P1.A6 (D+)
- new net: D13.3 (K), P1.A7 (D-)
- new net: D4.1 (K), R8.1
- new net: D3.1 (K), R7.1
- no-connect marks 30 -> 33
Other:
- note added: "Test Points"
- moved on the sheet: C14, Q1, Q2, R11, R12, R2, SW1, U9
