File: PCB_Files/watch.kicad_pcb (KiCad board)
At the start: 4 copper layers, 41 x 41 mm, 121 parts, among them J1 Conn_01x02_Pin, J2 Conn_01x14_MountingPin, J3 Conn_01x02_Pin, P1 USB_C_Plug_USB2.0, Q1 BC847, Q2 BC847, Q4 BSS138, Q5 BSS138, Q8 BC847, SW1 SW_Push, SW2 SW_Push, U1 APS6404L-3SQRx-ZR, U10 LSM6DS3, U11 MAX-M10S, U12 MCP1700x-120xxMB, U13 DRV2605LDGS, U14 TLV75533PDBV, U15 BQ24074RGT, U2 ESP32-PICO-D4, U3 CP2102N-Axx-xQFN28, U7 MAX30105EFD_T, U8 W25Q128JVS, U9 BMP388

Commit message: Made changes in schematic and routing
Parts:
- removed C5: 8pF, Capacitor_SMD:C_0603_1608Metric
- removed C6: 10pF, Capacitor_SMD:C_0603_1608Metric
- removed R7: 10k, Resistor_SMD:R_0603_1608Metric
- removed U8: W25Q128JVS, footprints:SOIC-8_5.23x5.23mm_P1.27mm
- removed XTAL1: ECS-400-10-37B2-CKY-TR, footprints:ECX-1637B2_ECS
- added U4: W25Q128JVP, Package_SON:WSON-8-1EP_6x5mm_P1.27mm_EP3.4x4.3mm, B.Cu at (145.3, 92.2)
- U1: moved to F.Cu
- moved TP1 9.87 mm to (133.3, 96.0)
- moved TP2 9.87 mm to (131.3, 96.0)
- moved TP7 9.87 mm to (132.0, 93.9)
- moved C21 8.07 mm to (154.2, 100.5), turned to 180 degrees
- moved C29 7.02 mm to (153.8, 102.1), turned to 180 degrees
- moved U1 6.18 mm to (146.4, 97.2)
- moved C8 5.81 mm to (132.6, 98.1), turned to 90 degrees
- moved C10 5.21 mm to (135.1, 94.1)
- moved C12 5.21 mm to (135.1, 92.6)
- moved C9 5.21 mm to (135.1, 95.6)
- moved C35 4.35 mm to (134.5, 91.8)
- moved L2 4.35 mm to (136.0, 91.8)
- moved U2 4.15 mm to (139.3, 97.4)
- moved C39 3.87 mm to (141.1, 97.7)
- moved R8 3.84 mm to (135.1, 105.6)
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Connections:
- U1 pad 2: /VSPIQ -> /VSPIQ_RAM
- U1 pad 3: /VSPIWP -> /VSPIWP_RAM
- U1 pad 5: /VSPID -> /VSPID_RAM
- U1 pad 6: /VSPICLK -> /VSPICLK_RAM
- U1 pad 7: /VSPIHD -> /VSPIHD_RAM
- U2 pad 15: unconnected-(U2-IO26-Pad15) -> /MISO
- U2 pad 24: /CE -> /MOSI
- U2 pad 28: /MISO -> /VSPIWP_RAM
- U2 pad 29: /MOSI -> /CE
- U2 pad 30: unconnected-(U2-CMD-Pad30) -> /VSPIHD_RAM
- U2 pad 31: unconnected-(U2-CLK-Pad31) -> /VSPICLK_RAM
- U2 pad 32: unconnected-(U2-SD0-Pad32) -> /VSPIQ_RAM
- U2 pad 33: unconnected-(U2-SD1-Pad33) -> /VSPID_RAM
- U2 pad 44: /XTAL_N -> unconnected-(U2-XTAL_N-Pad44)
- U2 pad 45: /XTAL_P -> unconnected-(U2-XTAL_P-Pad45)
Routing:
- net /INTR1_IMU: track 0.00 -> 21.5 mm, vias 0 -> 2
- net /EN: track 35.1 -> 55.7 mm, vias 2 -> 3
- net /CS: track 0.00 -> 15.8 mm, vias 0 -> 2
- net /CTP_INT: track 0.00 -> 13.0 mm, vias 0 -> 2
- net /LEDK: track 0.00 -> 12.4 mm, vias 0 -> 2
- net /SCL_i2c: track 22.1 -> 32.9 mm
- net /MOSI: track 0.00 -> 10.2 mm, vias 0 -> 2
- net /SCL: track 0.00 -> 7.91 mm
- net /SDA: track 20.3 -> 27.7 mm, vias 3 -> 4
- net /BL_PWM: track 0.00 -> 6.86 mm
- net /VSPIQ_RAM: track 0.00 -> 6.17 mm, vias 0 -> 2
- net /VSPICLK_RAM: track 0.00 -> 6.02 mm
- net /VSPID_RAM: track 0.00 -> 5.90 mm
- net /VSPIWP_RAM: track 0.00 -> 5.23 mm
- net /XTAL_N: track 4.54 -> 0.00 mm
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
Commit message: First commit of restarting layout
Parts:
- C10, C12, C17, C18, C19, C21, C23, C29, C33, C34, C37, C39, C8, C9, D2, D7, D9, L1, Q4, Q5, R10, R18, R19, R20, R21, R22, R23, R24, R25, R26, R27, R31, R34, R35, R39, R4, R40, R41, R42, R43, R9, U15, U4, U7, U9: moved to F.Cu
- moved R19 55.3 mm to (143.5, 52.9)
- moved J2 54.1 mm to (163.8, 64.8), turned to 0 degrees
- moved R20 52.8 mm to (143.5, 55.4), turned to 0 degrees
- moved J3 52.8 mm to (156.5, 63.3), turned to 0 degrees
- moved R22 52.5 mm to (143.5, 60.4), turned to 0 degrees
- moved C32 51.4 mm to (135.5, 57.9)
- moved C30 51.2 mm to (135.5, 52.9)
- moved C17 50.7 mm to (131.5, 55.4), turned to 0 degrees
- moved R1 50.6 mm to (139.5, 55.4)
- moved C26 49.2 mm to (131.5, 75.4), turned to 0 degrees
- moved R33 48.6 mm to (147.5, 52.9), turned to 0 degrees
- moved C19 48.4 mm to (131.5, 60.4), turned to 0 degrees
- moved R23 48.1 mm to (143.5, 62.9), turned to 0 degrees
- moved C31 47.9 mm to (135.5, 55.4), turned to 0 degrees
- moved R36 47.9 mm to (147.5, 60.4), turned to 0 degrees
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Connections:
- Q8 pad 2: GND -> unconnected-(Q8-E-Pad2)
- R36 pad 2: /LEDK -> unconnected-(R36-Pad2)
- R37 pad 1: /BL_PWM -> unconnected-(R37-Pad1)
Routing:
- net GND: track 139.7 -> 0.00 mm, vias 29 -> 0
- net /3V3: track 136.9 -> 0.00 mm, vias 6 -> 0
- net /EN: track 55.7 -> 0.00 mm, vias 3 -> 0
- net /D+: track 44.2 -> 0.00 mm, vias 2 -> 0
- net /1.8V: track 43.0 -> 0.00 mm, vias 3 -> 0
- net /D-: track 37.7 -> 0.00 mm, vias 2 -> 0
- net /SCL_i2c: track 32.9 -> 0.00 mm, vias 3 -> 0
- net /GPIO0: track 30.6 -> 0.00 mm, vias 2 -> 0
- net /SDA: track 27.7 -> 0.00 mm, vias 4 -> 0
- net /LV_SDA: track 25.9 -> 0.00 mm, vias 2 -> 0
- net /INTR1_IMU: track 21.5 -> 0.00 mm, vias 2 -> 0
- net /VBUS: track 20.1 -> 0.00 mm, vias 3 -> 0
- net /Batt+: track 17.8 -> 0.00 mm, vias 2 -> 0
- net /LV_SCL: track 16.7 -> 0.00 mm, vias 2 -> 0
- net /CS: track 15.8 -> 0.00 mm, vias 2 -> 0
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- removed copper zone on In1.Cu, net GND
Other:
- board outline removed

Commit message: Did routing of ESP, USB, USB-to-TTL, RAM, Flash, Osscilator & PMIC
Parts:
- moved J3 180.8 mm to (34.0, 196.2)
- moved C22 170.7 mm to (283.2, 143.6)
- moved R2 165.3 mm to (283.3, 139.4)
- moved C14 164.6 mm to (282.4, 136.0)
- moved C27 151.9 mm to (280.8, 105.9)
- moved C28 151.9 mm to (280.8, 108.4)
- moved C30 151.8 mm to (242.1, 160.9)
- moved C31 151.8 mm to (242.1, 163.4)
- moved R32 151.5 mm to (283.1, 141.8)
- moved SW1 149.7 mm to (278.5, 139.3)
- moved SW2 149.7 mm to (278.5, 143.7)
- moved R11 149.4 mm to (278.2, 133.8)
- moved R12 149.4 mm to (278.2, 136.3)
- moved Q1 146.4 mm to (271.9, 137.9)
- moved Q2 146.4 mm to (271.9, 142.3)
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Routing:
- net /3V3: track 0.00 -> 92.3 mm, vias 0 -> 9
- net GND: track 0.00 -> 52.1 mm, vias 0 -> 19
- net /CS_ROM: track 0.00 -> 26.0 mm, vias 0 -> 2
- net /Batt+: track 0.00 -> 21.0 mm, vias 0 -> 3
- net /VSPIHD: track 0.00 -> 18.5 mm, vias 0 -> 2
- net /D+: track 0.00 -> 17.2 mm, vias 0 -> 2
- net /VSPIQ: track 0.00 -> 16.2 mm, vias 0 -> 2
- net /D-: track 0.00 -> 16.2 mm, vias 0 -> 2
- net /BAT+: track 0.00 -> 14.8 mm
- net /VSPIWP: track 0.00 -> 14.6 mm, vias 0 -> 2
- net /VBUS: track 0.00 -> 14.6 mm, vias 0 -> 2
- net /EXT_5V: track 0.00 -> 13.4 mm
- net Net-(P1-CC): track 0.00 -> 13.3 mm
- net /VSPICLK: track 0.00 -> 12.5 mm, vias 0 -> 2
- net /VSPID: track 0.00 -> 10.9 mm, vias 0 -> 2
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- added copper zone on B.Cu, net GND
Other:
- board outline added: 107.2 x 60.1 mm
- copper layers 4 -> 2

Commit message: Restarted routing
Parts:
- removed J2: Conn_01x14_MountingPin, footprints:HRS_FH34SRJ-14S-0.5SH_50_
- added JP2: SolderJumper_2_Open, Resistor_SMD:R_0402_1005Metric, F.Cu at (91.3, 87.3)
- moved C28 188.1 mm to (95.6, 75.3), turned to -90 degrees
- moved C27 184.6 mm to (99.2, 72.5), turned to 180 degrees
- moved U9 182.8 mm to (100.6, 59.4), turned to 90 degrees
- moved U10 182.7 mm to (99.1, 76.2), turned to 180 degrees
- moved U12 181.7 mm to (86.3, 77.1), turned to 180 degrees
- moved D4 181.2 mm to (92.5, 77.1)
- moved C30 180.1 mm to (82.9, 76.7), turned to 90 degrees
- moved C31 174.0 mm to (92.4, 74.7)
- moved TP1 173.3 mm to (139.3, 26.2)
- moved TP2 173.3 mm to (139.3, 29.2)
- moved TP3 173.3 mm to (142.3, 26.2)
- moved TP4 173.3 mm to (142.3, 29.2)
- moved TP5 173.3 mm to (145.4, 26.2)
- moved TP6 173.3 mm to (145.4, 29.2)
- moved TP7 173.3 mm to (148.4, 26.2)
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Connections:
- Q8 pad 2: unconnected-(Q8-E-Pad2) -> GND
- R36 pad 2: unconnected-(R36-Pad2) -> /LEDK
- R37 pad 1: unconnected-(R37-Pad1) -> Net-(Q8-B)
- R37 pad 2: Net-(Q8-B) -> /BL_PWM
- U2 pad 25: /CE -> unconnected-(U2-IO16-Pad25)
- U4 pad 8: /3V3 -> Net-(JP2-A)
Routing:
- net /3V3: track 92.3 -> 3.30 mm, vias 9 -> 0
- net /GPIO0: track 0.00 -> 31.9 mm, vias 0 -> 2
- net /EN: track 0.00 -> 26.9 mm, vias 0 -> 2
- net /Batt+: track 21.0 -> 0.00 mm, vias 3 -> 0
- net /DTR: track 0.00 -> 19.3 mm, vias 0 -> 2
- net GND: track 52.1 -> 70.3 mm, vias 19 -> 27
- net /RTS: track 0.00 -> 13.6 mm, vias 0 -> 2
- net /SCL: track 0.00 -> 11.2 mm, vias 0 -> 2
- net /LNA_IN: track 1.48 -> 11.4 mm
- net /VSPIHD: track 18.5 -> 10.2 mm
- net /VSPID: track 10.9 -> 3.03 mm, vias 2 -> 0
- net Net-(C8-Pad1): track 7.79 -> 0.00 mm
- net Net-(AE2-A): track 4.13 -> 11.7 mm
- net /VSPICLK: track 12.5 -> 4.94 mm, vias 2 -> 0
- net /VSPIQ: track 16.2 -> 8.63 mm
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- added copper zone on F.Cu, net /1.8V
- added copper zone on F.Cu, net /32K_P
- added copper zone on F.Cu, net /3V3
- added copper zone on F.Cu, net /BAT+
- added copper zone on F.Cu, net /Batt+
- added copper zone on F.Cu, net GND
Other:
- board size 107.2 x 60.1 mm -> 60 x 60 mm
